File: SmartSwitch3.sch (EAGLE design)
At the start: 26 parts

Commit message: Change Jumper
Parts:
- removed LEDS: (no value), adafruit:PINHD-1X3
- added JP6: (no value), SparkFun-Connectors:M03PTH
Connections:
- net N$28: now also JP6.3; no longer LEDS.1
- net N$29: now also JP6.1; no longer LEDS.3
- net N$30: now also JP6.2; no longer LEDS.2
Changed lines of the file:
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@@
 <part name="OUT" library="wirepad" deviceset="2,15/1,0" device=""/>
 <part name="MCP23017" library="adafruit" deviceset="MCP23017" device="SP"/>
-<part name="LEDS" library="adafruit" deviceset="PINHD-1X3" device=""/>
 <part name="R1" library="SparkFun-Passives" deviceset="RESISTOR" device="PTH-1/2W"/>
 <part name="R2" library="SparkFun-Passives" deviceset="RESISTOR" device="PTH-1/2W"/>
@@
 <part name="JP3" library="SparkFun-Connectors" deviceset="M02" device="PTH"/>
 <part name="JP7" library="SparkFun-Connectors" deviceset="M02" device="PTH"/>
+<part name="JP6" library="SparkFun-Connectors" deviceset="M03" device="PTH"/>
 </parts>
 <sheets>
@@
 <instance part="OUT" gate="1" x="-38.1" y="50.546"/>
 <instance part="MCP23017" gate="G$1" x="109.22" y="30.48"/>
-<instance part="LEDS" gate="A" x="13.97" y="41.91"/>
 <instance part="R1" gate="G$1" x="81.28" y="59.69"/>
 <instance part="R2" gate="G$1" x="81.28" y="54.61"/>
@@
 <instance part="JP3" gate="G$1" x="130.556" y="27.94" rot="R180"/>
 <instance part="JP7" gate="G$1" x="186.944" y="35.56" rot="R180"/>
+<instance part="JP6" gate="G$1" x="3.81" y="41.91"/>
 </instances>
 <busses>
@@
 <pinref part="JP2" gate="G$1" pin="2"/>
 <wire x1="67.31" y1="58.42" x2="26.67" y2="58.42" width="0.1524" layer="91"/>
-<pinref part="LEDS" gate="A" pin="1"/>
 <wire x1="26.67" y1="58.42" x2="17.78" y2="58.42" width="0.1524" layer="91"/>
 <wire x1="11.43" y1="44.45" x2="22.86" y2="44.45" width="0.1524" layer="91"/>
@@
 <wire x1="26.67" y1="48.26" x2="26.67" y2="58.42" width="0.1524" layer="91"/>
 <junction x="26.67" y="58.42"/>
+<pinref part="JP6" gate="G$1" pin="3"/>
 </segment>
 </net>
 <net name="N$29" class="0">
 <segment>
-<pinref part="LEDS" gate="A" pin="3"/>
 <wire x1="11.43" y1="39.37" x2="11.43" y2="33.274" width="0.1524" layer="91"/>
 <wire x1="11.43" y1="33.274" x2="31.75" y2="20.32" width="0.1524" layer="91"/>
@@
 <wire x1="19.05" y1="7.62" x2="31.75" y2="20.32" width="0.1524" layer="91"/>
 <junction x="31.75" y="20.32"/>
+<pinref part="JP6" gate="G$1" pin="1"/>
 </segment>
 </net>
 <net name="N$30" class="0">
 <segment>
-<pinref part="LEDS" gate="A" pin="2"/>
 <wire x1="31.75" y1="45.72" x2="31.75" y2="41.91" width="0.1524" layer="91"/>
 <wire x1="31.75" y1="41.91" x2="11.43" y2="41.91" width="0.1524" layer="91"/>
@@
 <wire x1="30.48" y1="54.61" x2="30.48" y2="46.99" width="0.1524" layer="91"/>
 <wire x1="30.48" y1="46.99" x2="31.75" y2="45.72" width="0.1524" layer="91"/>
-</segment>
-</net>
+<pinref part="JP6" gate="G$1" pin="2"/>
+</segment>
+</net>
