File: SmartSwitch2.sch (EAGLE design)
At the start: 26 parts

Commit message: Change Jumper
Parts:
- removed LEDS: (no value), adafruit:PINHD-1X3
- added JP6: (no value), SparkFun-Connectors:M03PTH
Connections:
- net N$28: now also JP6.3; no longer LEDS.1
- net N$29: now also JP6.1; no longer LEDS.3
- net N$30: now also JP6.2; no longer LEDS.2
Changed lines of the file:
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@@
 <part name="OUT" library="wirepad" deviceset="2,15/1,0" device=""/>
 <part name="MCP23017" library="adafruit" deviceset="MCP23017" device="SP"/>
-<part name="LEDS" library="adafruit" deviceset="PINHD-1X3" device=""/>
 <part name="R1" library="SparkFun-Passives" deviceset="RESISTOR" device="PTH-1/2W"/>
 <part name="R2" library="SparkFun-Passives" deviceset="RESISTOR" device="PTH-1/2W"/>
@@
 <part name="JP3" library="SparkFun-Connectors" deviceset="M02" device="PTH"/>
 <part name="JP7" library="SparkFun-Connectors" deviceset="M02" device="PTH"/>
+<part name="JP6" library="SparkFun-Connectors" deviceset="M03" device="PTH"/>
 </parts>
 <sheets>
@@
 <instance part="OUT" gate="1" x="-38.1" y="50.546"/>
 <instance part="MCP23017" gate="G$1" x="109.22" y="30.48"/>
-<instance part="LEDS" gate="A" x="13.97" y="41.91"/>
 <instance part="R1" gate="G$1" x="81.28" y="59.69"/>
 <instance part="R2" gate="G$1" x="81.28" y="54.61"/>
@@
 <instance part="SWITCH" gate="1" x="-38.1" y="71.12"/>
 <instance part="JP2" gate="G$1" x="10.16" y="55.88"/>
-<instance part="JP1" gate="G$1" x="139.7" y="17.526" rot="R180"/>
+<instance part="JP1" gate="G$1" x="139.954" y="17.78" rot="R180"/>
 <instance part="JP3" gate="G$1" x="130.556" y="27.94" rot="R180"/>
 <instance part="JP7" gate="G$1" x="186.944" y="35.56" rot="R180"/>
+<instance part="JP6" gate="G$1" x="3.81" y="41.91"/>
 </instances>
 <busses>
@@
 <pinref part="JP2" gate="G$1" pin="2"/>
 <wire x1="67.31" y1="58.42" x2="26.67" y2="58.42" width="0.1524" layer="91"/>
-<pinref part="LEDS" gate="A" pin="1"/>
 <wire x1="26.67" y1="58.42" x2="17.78" y2="58.42" width="0.1524" layer="91"/>
 <wire x1="11.43" y1="44.45" x2="22.86" y2="44.45" width="0.1524" layer="91"/>
@@
 <wire x1="26.67" y1="48.26" x2="26.67" y2="58.42" width="0.1524" layer="91"/>
 <junction x="26.67" y="58.42"/>
+<pinref part="JP6" gate="G$1" pin="3"/>
 </segment>
 </net>
 <net name="N$29" class="0">
 <segment>
-<pinref part="LEDS" gate="A" pin="3"/>
 <wire x1="11.43" y1="39.37" x2="11.43" y2="33.274" width="0.1524" layer="91"/>
 <wire x1="11.43" y1="33.274" x2="31.75" y2="20.32" width="0.1524" layer="91"/>
@@
 <wire x1="19.05" y1="7.62" x2="31.75" y2="20.32" width="0.1524" layer="91"/>
 <junction x="31.75" y="20.32"/>
+<pinref part="JP6" gate="G$1" pin="1"/>
 </segment>
 </net>
 <net name="N$30" class="0">
 <segment>
-<pinref part="LEDS" gate="A" pin="2"/>
 <wire x1="31.75" y1="45.72" x2="31.75" y2="41.91" width="0.1524" layer="91"/>
 <wire x1="31.75" y1="41.91" x2="11.43" y2="41.91" width="0.1524" layer="91"/>
@@
 <wire x1="30.48" y1="54.61" x2="30.48" y2="46.99" width="0.1524" layer="91"/>
 <wire x1="30.48" y1="46.99" x2="31.75" y2="45.72" width="0.1524" layer="91"/>
-</segment>
-</net>
+<pinref part="JP6" gate="G$1" pin="2"/>
+</segment>
+</net>

Commit message: Resistors
Parts:
- added R3, R4, R5, R6, R7, R8: (no value), SparkFun-Resistors:RESISTORPTH-1/4W
- R1, R2: device SparkFun-Passives:RESISTORPTH-1/2W -> SparkFun-Resistors:RESISTORPTH-1/4W
Connections:
- new net N$20: MCP23017.GPB2, R3.1
- new net N$21: JP1.1, R3.2
- new net N$22: JP1.2, R4.2
- new net N$23: JP1.3, R5.2
- new net N$24: JP1.4, R6.2
- new net N$25: JP1.5, R7.2
- new net N$45: JP1.6, R8.2
- new net N$52: MCP23017.GPB7, R8.1
- new net N$53: MCP23017.GPB6, R7.1
- new net N$54: MCP23017.GPB5, R6.1
- new net N$55: MCP23017.GPB4, R5.1
- new net N$56: MCP23017.GPB3, R4.1
- net N$28: now also MCP23017.VDD
- net N$33: now also R2.2
- net N$49: no longer MCP23017.VDD
- net N$51: no longer R2.2
Other:
- moved on the sheet: JP1
Changed lines of the file:
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@@
 <part name="OUT" library="wirepad" deviceset="2,15/1,0" device=""/>
 <part name="MCP23017" library="adafruit" deviceset="MCP23017" device="SP"/>
-<part name="R1" library="SparkFun-Passives" deviceset="RESISTOR" device="PTH-1/2W"/>
-<part name="R2" library="SparkFun-Passives" deviceset="RESISTOR" device="PTH-1/2W"/>
+<part name="R1" library="SparkFun-Resistors" deviceset="RESISTOR" device="PTH-1/4W"/>
+<part name="R2" library="SparkFun-Resistors" deviceset="RESISTOR" device="PTH-1/4W"/>
 <part name="BUTTONPAD" library="SparkFun-Connectors" deviceset="M06" device="SILK_FEMALE_PTH"/>
 <part name="SPARK" library="Spark" deviceset="SPARK_CORE" device="CORE"/>
@@
 <part name="SWITCH" library="wirepad" deviceset="2,15/1,0" device=""/>
 <part name="JP2" library="SparkFun-Connectors" deviceset="M02" device="PTH"/>
-<part name="JP1" library="SparkFun-Connectors" deviceset="M06" device="SILK_FEMALE_PTH"/>
 <part name="JP3" library="SparkFun-Connectors" deviceset="M02" device="PTH"/>
 <part name="JP7" library="SparkFun-Connectors" deviceset="M02" device="PTH"/>
 <part name="JP6" library="SparkFun-Connectors" deviceset="M03" device="PTH"/>
+<part name="R3" library="SparkFun-Resistors" deviceset="RESISTOR" device="PTH-1/4W"/>
+<part name="R4" library="SparkFun-Resistors" deviceset="RESISTOR" device="PTH-1/4W"/>
+<part name="R5" library="SparkFun-Resistors" deviceset="RESISTOR" device="PTH-1/4W"/>
+<part name="R6" library="SparkFun-Resistors" deviceset="RESISTOR" device="PTH-1/4W"/>
+<part name="R7" library="SparkFun-Resistors" deviceset="RESISTOR" device="PTH-1/4W"/>
+<part name="R8" library="SparkFun-Resistors" deviceset="RESISTOR" device="PTH-1/4W"/>
+<part name="JP1" library="SparkFun-Connectors" deviceset="M06" device="SILK_FEMALE_PTH"/>
 </parts>
 <sheets>
@@
 <instance part="SWITCH" gate="1" x="-38.1" y="71.12"/>
 <instance part="JP2" gate="G$1" x="10.16" y="55.88"/>
-<instance part="JP1" gate="G$1" x="139.954" y="17.78" rot="R180"/>
 <instance part="JP3" gate="G$1" x="130.556" y="27.94" rot="R180"/>
 <instance part="JP7" gate="G$1" x="186.944" y="35.56" rot="R180"/>
 <instance part="JP6" gate="G$1" x="3.81" y="41.91"/>
+<instance part="R3" gate="G$1" x="140.716" y="22.86"/>
+<instance part="R4" gate="G$1" x="140.208" y="20.32"/>
+<instance part="R5" gate="G$1" x="139.954" y="17.78"/>
+<instance part="R6" gate="G$1" x="139.446" y="15.24"/>
+<instance part="R7" gate="G$1" x="140.208" y="12.7"/>
+<instance part="R8" gate="G$1" x="140.208" y="10.16"/>
+<instance part="JP1" gate="G$1" x="151.384" y="17.78" rot="R180"/>
 </instances>
 <busses>
@@
 <junction x="26.67" y="58.42"/>
 <pinref part="JP6" gate="G$1" pin="3"/>
+<pinref part="MCP23017" gate="G$1" pin="VDD"/>
+<wire x1="96.52" y1="50.8" x2="91.44" y2="50.8" width="0.1524" layer="91"/>
+<junction x="91.44" y="50.8"/>
 </segment>
 </net>
@@
 <wire x1="57.15" y1="0" x2="67.31" y2="0" width="0.1524" layer="91"/>
 <junction x="67.31" y="0"/>
+<wire x1="106.68" y1="54.61" x2="106.68" y2="38.1" width="0.1524" layer="91"/>
+<pinref part="R2" gate="G$1" pin="2"/>
+<wire x1="86.36" y1="54.61" x2="106.68" y2="54.61" width="0.1524" layer="91"/>
+<wire x1="96.52" y1="27.94" x2="106.68" y2="38.1" width="0.1524" layer="91"/>
+<junction x="96.52" y="27.94"/>
 </segment>
 </net>
@@
 <wire x1="67.31" y1="45.72" x2="66.04" y2="45.72" width="0.1524" layer="91"/>
 <wire x1="66.04" y1="45.72" x2="55.88" y2="35.56" width="0.1524" layer="91"/>
-<pinref part="MCP23017" gate="G$1" pin="VDD"/>
-<wire x1="67.31" y1="45.72" x2="91.44" y2="45.72" width="0.1524" layer="91"/>
-<wire x1="91.44" y1="45.72" x2="96.52" y2="50.8" width="0.1524" layer="91"/>
-<junction x="67.31" y="45.72"/>
 </segment>
 </net>
@@
 <net name="N$51" class="0">
 <segment>
-<pinref part="R2" gate="G$1" pin="2"/>
-<wire x1="86.36" y1="54.61" x2="106.68" y2="54.61" width="0.1524" layer="91"/>
-<wire x1="106.68" y1="54.61" x2="106.68" y2="40.64" width="0.1524" layer="91"/>
 <pinref part="MCP23017" gate="G$1" pin="INTA"/>
 <wire x1="67.31" y1="10.16" x2="96.52" y2="40.64" width="0.1524" layer="91"/>
 <pinref part="SPARK" gate="G$1" pin="D3"/>
-<wire x1="106.68" y1="40.64" x2="96.52" y2="40.64" width="0.1524" layer="91"/>
-<junction x="96.52" y="40.64"/>
 <pinref part="JP5" gate="G$1" pin="4"/>
 <wire x1="55.88" y1="17.78" x2="59.69" y2="13.97" width="0.1524" layer="91"/>
@@
 </segment>
 </net>
+<net name="N$20" class="0">
+<segment>
+<pinref part="MCP23017" gate="G$1" pin="GPB2"/>
+<pinref part="R3" gate="G$1" pin="1"/>
+<wire x1="121.92" y1="22.86" x2="135.636" y2="22.86" width="0.1524" layer="91"/>
+</segment>
+</net>
+<net name="N$21" class="0">
+<segment>
+<pinref part="R3" gate="G$1" pin="2"/>
+<wire x1="145.796" y1="22.86" x2="146.304" y2="22.86" width="0.1524" layer="91"/>
+<pinref part="JP1" gate="G$1" pin="1"/>
+</segment>
+</net>
+<net name="N$22" class="0">
+<segment>
+<pinref part="R4" gate="G$1" pin="2"/>
+<wire x1="145.288" y1="20.32" x2="146.304" y2="20.32" width="0.1524" layer="91"/>
+<pinref part="JP1" gate="G$1" pin="2"/>
+</segment>
+</net>
+<net name="N$23" class="0">
+<segment>
+<pinref part="R5" gate="G$1" pin="2"/>
+<wire x1="145.034" y1="17.78" x2="146.304" y2="17.78" width="0.1524" layer="91"/>
+<pinref part="JP1" gate="G$1" pin="3"/>
+</segment>
+</net>
+<net name="N$24" class="0">
+<segment>
+<pinref part="R6" gate="G$1" pin="2"/>
+<wire x1="144.526" y1="15.24" x2="146.304" y2="15.24" width="0.1524" layer="91"/>
+<pinref part="JP1" gate="G$1" pin="4"/>
+</segment>
+</net>
+<net name="N$25" class="0">
+<segment>
+<pinref part="R7" gate="G$1" pin="2"/>
+<wire x1="145.288" y1="12.7" x2="146.304" y2="12.7" width="0.1524" layer="91"/>
+<pinref part="JP1" gate="G$1" pin="5"/>
+</segment>
+</net>
+<net name="N$45" class="0">
+<segment>
+<pinref part="R8" gate="G$1" pin="2"/>
+<wire x1="145.288" y1="10.16" x2="146.304" y2="10.16" width="0.1524" layer="91"/>
+<pinref part="JP1" gate="G$1" pin="6"/>
+</segment>
+</net>
+<net name="N$52" class="0">
+<segment>
+<pinref part="MCP23017" gate="G$1" pin="GPB7"/>
+<pinref part="R8" gate="G$1" pin="1"/>
+<wire x1="121.92" y1="10.16" x2="135.128" y2="10.16" width="0.1524" layer="91"/>
+</segment>
+</net>
+<net name="N$53" class="0">
+<segment>
+<pinref part="R7" gate="G$1" pin="1"/>
+<pinref part="MCP23017" gate="G$1" pin="GPB6"/>
+<wire x1="135.128" y1="12.7" x2="121.92" y2="12.7" width="0.1524" layer="91"/>
+</segment>
+</net>
+<net name="N$54" class="0">
+<segment>
+<pinref part="MCP23017" gate="G$1" pin="GPB5"/>
+<pinref part="R6" gate="G$1" pin="1"/>
+<wire x1="121.92" y1="15.24" x2="134.366" y2="15.24" width="0.1524" layer="91"/>
+</segment>
+</net>
+<net name="N$55" class="0">
+<segment>
+<pinref part="R5" gate="G$1" pin="1"/>
+<pinref part="MCP23017" gate="G$1" pin="GPB4"/>
+<wire x1="134.874" y1="17.78" x2="121.92" y2="17.78" width="0.1524" layer="91"/>
+</segment>
+</net>
+<net name="N$56" class="0">
+<segment>
+<pinref part="MCP23017" gate="G$1" pin="GPB3"/>
+<pinref part="R4" gate="G$1" pin="1"/>
+<wire x1="121.92" y1="20.32" x2="135.128" y2="20.32" width="0.1524" layer="91"/>
+</segment>
+</net>
